Commit message: two

File: src/articubot_one/description/arm_robot.xacro (robot description, xacro)
@@ -1,4 +1,4 @@
 <?xml version="1.0"?>
-<robot xmlns:xacro="http://www.ros.org/wiki/xacro">
+<robot xmlns:xacro="http://www.ros.org/wiki/xacro" name="articubot">
     <xacro:include filename="inertial_macros.xacro"/>
     <xacro:property name="arm_base_length" value="0.1" />
@@ -157,9 +157,9 @@
                                 xyz="0 0 ${hand_length / 2.0}" rpy="0 0 0" />
     </link>
-    <joint name="mobile_base_arm_joint" type="fixed">
+    <!-- <joint name="mobile_base_arm_joint" type="fixed">
         <parent link="chassis" />
         <child link="arm_base_link" />
         <origin xyz="${8*chassis_length / 9.0} 0 ${chassis_height}" rpy="0 0 0" />
-    </joint>
+    </joint> -->
     <joint name="arm_base_forearm_joint" type="revolute">
         <parent link="arm_base_link" />

File: src/articubot_one/description/robot.urdf.xacro (robot description, xacro)
@@ -16,3 +16,8 @@
     <!-- <xacro:include filename="depth_camera.xacro" /> -->
     <xacro:include filename="face.xacro" />
+    <joint name="mobile_base_arm_joint" type="fixed">
+        <parent link="chassis" />
+        <child link="arm_base_link" />
+        <origin xyz="${8*chassis_length / 9.0} 0 ${chassis_height}" rpy="0 0 0" />
+    </joint>
 </robot>

Commit message: add action

File: src/articubot_one/description/arm_robot.xacro (robot description, xacro)
@@ -157,9 +157,9 @@
                                 xyz="0 0 ${hand_length / 2.0}" rpy="0 0 0" />
     </link>
-    <!-- <joint name="mobile_base_arm_joint" type="fixed">
+    <joint name="mobile_base_arm_joint" type="fixed">
         <parent link="chassis" />
         <child link="arm_base_link" />
         <origin xyz="${8*chassis_length / 9.0} 0 ${chassis_height}" rpy="0 0 0" />
-    </joint> -->
+    </joint>
     <joint name="arm_base_forearm_joint" type="revolute">
         <parent link="arm_base_link" />

File: src/articubot_one/description/depth_camera.xacro (robot description, xacro)
@@ -2,7 +2,7 @@
 <robot xmlns:xacro="http://www.ros.org/wiki/xacro" >
     <joint name="camera_joint" type="fixed">
-        <parent link="chassis"/>
+        <parent link="claw_support"/>
         <child link="camera_link"/>
-        <origin xyz="0.305 0 0.08" rpy="0 0 0"/>
+        <origin xyz="0.05 0 0.08" rpy="0 0 0"/>
     </joint>
     <link name="camera_link">

File: src/articubot_one/description/robot.urdf.xacro (robot description, xacro)
@@ -6,5 +6,5 @@
     <xacro:include filename="arm_robot.xacro" />
     <xacro:include filename="inertial_macros.xacro" />
-    <xacro:include filename="camera.xacro" />
+    <!-- <xacro:include filename="camera.xacro" /> -->
     <xacro:if value="$(arg use_ros2_control)">
         <xacro:include filename="ros2_control.xacro" />
@@ -14,10 +14,10 @@
     </xacro:unless>
     <xacro:include filename="lidar.xacro" />
-    <!-- <xacro:include filename="depth_camera.xacro" /> -->
+    <xacro:include filename="depth_camera.xacro" />
     <xacro:include filename="face.xacro" />
-    <joint name="mobile_base_arm_joint" type="fixed">
+    <!-- <joint name="mobile_base_arm_joint" type="fixed">
         <parent link="chassis" />
         <child link="arm_base_link" />
         <origin xyz="${8*chassis_length / 9.0} 0 ${chassis_height}" rpy="0 0 0" />
-    </joint>
+    </joint> -->
 </robot>
